File: USB_inspection-light.sch (KiCad schematic (older format))
At the start: 22 parts, among them CON1 USB-MINI-B, IC1 MADW__ATTINY13-MM, Q1 MOSFET_N, SW1 SW_PUSH, SW2 SW_PUSH

Commit message: Added 100k pull-down resistor to mosfet gate.
Purpose: prevent LED flash on power-up.
Parts:
- added R10: 100k, symbol R
Connections:
- net GND: now also R10.1
- net at Q1.1 (G), R7.2: now also R10.2
Changed lines of the file:
@@
 Sheet 1 1
 Title "USB inspection light"
-Date "23 Feb 2014"
-Rev "0.10"
+Date "06 May 2014"
+Rev "0.20"
 Comp "2014 - blog.spitzenpfeil.org"
 Comment1 ""
@@
 U 1 1 51640F23
 P 6600 2650
-F 0 "R7" V 6680 2650 50  0000 C CNN
+F 0 "R7" V 6500 2650 50  0000 C CNN
 F 1 "150R" V 6600 2650 50  0000 C CNN
 F 2 "" H 6600 2650 60  0000 C CNN
@@
 P 6950 2650
 F 0 "Q1" H 7150 2940 60  0000 R CNN
-F 1 "MOSFET_N" H 7150 2550 60  0000 R CNN
+F 1 "MOSFET_N" H 7800 2650 60  0000 R CNN
 F 2 "~" H 6950 2650 60  0000 C CNN
 F 3 "~" H 6950 2650 60  0000 C CNN
@@
 	7250 2750 7250 3450
 $Comp
-L GND #PWR02
+L GND #PWR01
 U 1 1 51641142
 P 7250 3450
-F 0 "#PWR02" H 7250 3450 30  0001 C CNN
+F 0 "#PWR01" H 7250 3450 30  0001 C CNN
 F 1 "GND" H 7250 3380 30  0001 C CNN
 F 2 "" H 7250 3450 60  0000 C CNN
@@
 $EndComp
 $Comp
-L +5V #PWR03
+L +5V #PWR02
 U 1 1 516412DB
 P 5050 3550
-F 0 "#PWR03" H 5050 3640 20  0001 C CNN
+F 0 "#PWR02" H 5050 3640 20  0001 C CNN
 F 1 "+5V" H 5050 3640 30  0000 C CNN
 F 2 "" H 5050 3550 60  0000 C CNN
@@
 	5050 3550 5050 3700
 $Comp
-L GND #PWR04
+L GND #PWR03
 U 1 1 51641344
 P 5050 4300
-F 0 "#PWR04" H 5050 4300 30  0001 C CNN
+F 0 "#PWR03" H 5050 4300 30  0001 C CNN
 F 1 "GND" H 5050 4230 30  0001 C CNN
 F 2 "" H 5050 4300 60  0000 C CNN
@@
 $EndComp
 $Comp
-L GND #PWR05
+L GND #PWR04
 U 1 1 5164148D
 P 1500 4800
-F 0 "#PWR05" H 1500 4800 30  0001 C CNN
+F 0 "#PWR04" H 1500 4800 30  0001 C CNN
 F 1 "GND" H 1500 4730 30  0001 C CNN
 F 2 "" H 1500 4800 60  0000 C CNN
@@
 	4150 5000 4450 5000
 $Comp
-L GND #PWR06
+L GND #PWR05
 U 1 1 516419E6
 P 4450 5150
-F 0 "#PWR06" H 4450 5150 30  0001 C CNN
+F 0 "#PWR05" H 4450 5150 30  0001 C CNN
 F 1 "GND" H 4450 5080 30  0001 C CNN
 F 2 "" H 4450 5150 60  0000 C CNN
@@
 $EndComp
 $Comp
-L +5V #PWR07
+L +5V #PWR06
 U 1 1 516419F5
 P 4450 4700
-F 0 "#PWR07" H 4450 4790 20  0001 C CNN
+F 0 "#PWR06" H 4450 4790 20  0001 C CNN
 F 1 "+5V" H 4450 4790 30  0000 C CNN
 F 2 "" H 4450 4700 60  0000 C CNN
@@
 NoConn ~ 2950 4050
 $Comp
-L GND #PWR08
+L GND #PWR07
 U 1 1 51644384
 P 3700 6050
-F 0 "#PWR08" H 3700 6050 30  0001 C CNN
+F 0 "#PWR07" H 3700 6050 30  0001 C CNN
 F 1 "GND" H 3700 5980 30  0001 C CNN
 F 2 "" H 3700 6050 60  0000 C CNN
@@
 $EndComp
 $Comp
-L +5V #PWR09
+L +5V #PWR08
 U 1 1 51644393
 P 3950 6050
-F 0 "#PWR09" H 3950 6140 20  0001 C CNN
+F 0 "#PWR08" H 3950 6140 20  0001 C CNN
 F 1 "+5V" H 3950 6140 30  0000 C CNN
 F 2 "" H 3950 6050 60  0000 C CNN
@@
 $EndComp
 $Comp
-L PWR_FLAG #FLG010
+L PWR_FLAG #FLG09
 U 1 1 516443A2
 P 3700 5850
-F 0 "#FLG010" H 3700 5945 30  0001 C CNN
+F 0 "#FLG09" H 3700 5945 30  0001 C CNN
 F 1 "PWR_FLAG" H 3700 6030 30  0000 C CNN
 F 2 "" H 3700 5850 60  0000 C CNN
@@
 $EndComp
 $Comp
-L PWR_FLAG #FLG011
+L PWR_FLAG #FLG010
 U 1 1 516443B1
 P 3950 5850
-F 0 "#FLG011" H 3950 5945 30  0001 C CNN
+F 0 "#FLG010" H 3950 5945 30  0001 C CNN
 F 1 "PWR_FLAG" H 3950 6030 30  0000 C CNN
 F 2 "" H 3950 5850 60  0000 C CNN
@@
 	4950 4050 4950 4150
 $Comp
-L +5V #PWR012
+L +5V #PWR011
 U 1 1 530A2B9B
 P 7250 850
-F 0 "#PWR012" H 7250 940 20  0001 C CNN
+F 0 "#PWR011" H 7250 940 20  0001 C CNN
 F 1 "+5V" H 7250 940 30  0000 C CNN
 F 2 "" H 7250 850 60  0000 C CNN
@@
 NoConn ~ 7850 5500
 $Comp
-L GND #PWR013
+L GND #PWR012
 U 1 1 530A2CCB
 P 6600 5600
-F 0 "#PWR013" H 6600 5600 30  0001 C CNN
+F 0 "#PWR012" H 6600 5600 30  0001 C CNN
 F 1 "GND" H 6600 5530 30  0001 C CNN
 F 2 "" H 6600 5600 60  0000 C CNN
@@
 $EndComp
 $Comp
-L +5V #PWR014
+L +5V #PWR013
 U 1 1 530A2CDF
 P 6600 4800
-F 0 "#PWR014" H 6600 4890 20  0001 C CNN
+F 0 "#PWR013" H 6600 4890 20  0001 C CNN
 F 1 "+5V" H 6600 4890 30  0000 C CNN
 F 2 "" H 6600 4800 60  0000 C CNN
@@
 Wire Wire Line
 	8750 2200 7250 2200
+$Comp
+L GND #PWR014
+U 1 1 53692EB8
+P 6900 3250
+F 0 "#PWR014" H 6900 3250 30  0001 C CNN
+F 1 "GND" H 6900 3180 30  0001 C CNN
+F 2 "" H 6900 3250 60  0000 C CNN
+F 3 "" H 6900 3250 60  0000 C CNN
+	1    6900 3250
+	1    0    0    -1
+$EndComp
+Wire Wire Line
+	6900 3200 6900 3250
+Wire Wire Line
+	6900 2650 6900 2700
+Connection ~ 6900 2650
+$Comp
+L R R10
+U 1 1 5369329D
+P 6900 2950
+F 0 "R10" H 6750 2950 50  0000 C CNN
+F 1 "100k" V 6907 2951 50  0000 C CNN
+F 2 "" V 6830 2950 30  0000 C CNN
+F 3 "" H 6900 2950 30  0000 C CNN
+	1    6900 2950
+	-1   0    0    1
+$EndComp
 $EndSCHEMATC
